File: MGA_02.kicad_pcb (KiCad board)
At the start: 2 copper layers, 100 x 28 mm, 22 parts, among them J1 Painel +, J2 Painel -, J3 VDD, J4 GND, J5 BAT +, J6 BAT -, J7 OUT-, J8 OUT+

Commit message: Correção do Conversor DC-DC
Routing:
- net Net-(D4-Pad2): track 6.04 -> 23.5 mm
- net Net-(C1-Pad1): track 34.4 -> 36.7 mm
